Commit message: urdf update - ur3 btw walls

File: ur3/pointing/urdf/robot.urdf.xacro (robot description, xacro)
@@ -1,4 +1,7 @@
 <?xml version="1.0"?>
 <robot xmlns:xacro="http://wiki.ros.org/xacro" name="ur3e" >
+  <material name="white02">
+    <color rgba="1 1 1 0.2"/>
+  </material>
   <!-- parameters -->
   <xacro:arg name="gazebo" default="false"
@@ -51,32 +54,111 @@
       <inertial>
         <mass value="200"/>
-        <origin xyz="0 0 0.45"/>
+	<origin xyz="0 0 0.44"/>
         <inertia ixx="50"  ixy="0"  ixz="0" iyy="50" iyz="0" izz="50" />
       </inertial>
+      <!-- table -->
       <visual>
-        <origin xyz="-0.45 0.0 0.44"/>
-        <geometry>
-	        <box size="1.15 0.75 0.855"/>
+	<origin xyz="0.0 -0.305 0.5"/>
+        <geometry>
+	        <box size="0.80 1 1"/>
         </geometry>
       </visual>
       <collision>
-        <origin xyz="-0.45 0.0 0.44"/>
-        <geometry>
-	        <box size="1.15 0.75 0.855"/>
-        </geometry>
-      </collision>
-     <visual>
-       <origin xyz="0 0 0.875"/>
-       <geometry>
-	        <box size="0.15 0.21 0.02"/>
-       </geometry>
-     </visual>
-     <collision>
-       <origin xyz="0 0 0.875"/>
-       <geometry>
-	        <box size="0.15 0.21 0.02"/>
+        <origin xyz="0.0 -0.305 0.5"/>
+        <geometry>
+	        <box size="0.80 1 1"/>
+        </geometry>
+      </collision>
+      <!-- support -->
+     <visual>
+       <origin xyz="0 0 1.01"/>
+       <geometry>
+	        <box size="0.16 0.16 0.02"/>
+       </geometry>
+     </visual>
+     <collision>
+       <origin xyz="0 0 1.01"/>
+       <geometry>
+	        <box size="0.16 0.16 0.02"/>
        </geometry>
      </collision>
     </link>
+    <link name="walls">
+     <!-- front wall -->
+     <visual>
+	<origin xyz="0.385 -0.305 0.37"/>
+        <geometry>
+	  <box size="0.03 1 0.74"/>
+        </geometry>
+	<material name="white02"/>
+     </visual>
+      <collision>
+       <origin xyz="0.385 -0.305 0.37"/>
+       <geometry>
+	 <box size="0.03 1 0.74"/>
+       </geometry>
+      </collision>
+      <!-- behind wall -->
+     <visual>
+	<origin xyz="-0.385 -0.305 0.37"/>
+        <geometry>
+	  <box size="0.03 1 0.74"/>
+        </geometry>
+	<material name="white02"/>
+     </visual>
+      <collision>
+       <origin xyz="-0.385 -0.305 0.37"/>
+       <geometry>
+	 <box size="0.03 1 0.74"/>
+       </geometry>
+      </collision>
+      <!-- left wall -->
+     <visual>
+	<origin xyz="0 -0.79 0.37"/>
+        <geometry>
+	  <box size="0.74 0.03 0.74"/>
+        </geometry>
+	<material name="white02"/>
+     </visual>
+      <collision>
+       <origin xyz="0 -0.79 0.37"/>
+       <geometry>
+	 <box size="0.74 0.03 0.74"/>
+       </geometry>
+      </collision>
+     <!-- right wall -->
+     <visual>
+	<origin xyz="0 0.185 0.37"/>
+        <geometry>
+	  <box size="0.74 0.03 0.74"/>
+        </geometry>
+	<material name="white02"/>
+     </visual>
+      <collision>
+       <origin xyz="0 0.185 0.37"/>
+       <geometry>
+	 <box size="0.74 0.03 0.74"/>
+       </geometry>
+      </collision>
+      <!-- above wall -->
+     <visual>
+	<origin xyz="0 -0.305 0.755"/>
+        <geometry>
+	  <box size="0.80 1 0.03"/>
+        </geometry>
+	<material name="white02"/>
+     </visual>
+      <collision>
+       <origin xyz="0 -0.305 0.75"/>
+       <geometry>
+	 <box size="0.80 1 0.03"/>
+       </geometry>
+     </collision>
+    </link>
+    <joint name="walls_joint" type="fixed">
+     <parent link="support_link" />
+     <child link = "walls" />
+      <origin xyz="0.0 0.0 1" rpy="0.0 0.0 0" />
+   </joint>
    <joint name="support_joint" type="fixed">
      <parent link="world" />
@@ -87,5 +169,5 @@
      <parent link="support_link" />
      <child link = "base_link" />
-      <origin xyz="0.0 0.0 0.885" rpy="0.0 0.0 -1.5707963" />
+      <origin xyz="0.0 0.0 1" rpy="0.0 0.0 -1.5707963" />
    </joint>
    <link name="collision_cylinder">

Commit message: remove pointing end-effector

File: ur3/pointing/urdf/robot.urdf.xacro (robot description, xacro)
@@ -84,5 +84,5 @@
      </collision>
     </link>
-    <link name="walls">
+     <link name="walls">
      <!-- front wall -->
      <visual>
@@ -156,5 +156,5 @@
      </collision>
     </link>
-    <joint name="walls_joint" type="fixed">
+<joint name="walls_joint" type="fixed">
      <parent link="support_link" />
      <child link = "walls" />
@@ -172,4 +172,10 @@
    </joint>
    <link name="collision_cylinder">
+     <visual>
+        <origin xyz="0 0 0" rpy="0 0 0"/>
+       <geometry>
+	 <cylinder radius="0.045" length="0.115"/>
+       </geometry>
+     </visual>
      <collision>
        <origin xyz="0 0 0" rpy="0 0 0"/>
@@ -184,109 +190,8 @@
      <origin xyz="0.0 0.0 0.05" rpy="0.0 0.0 ${pi/2.0}" />
    </joint>
-   <joint name="ee_fixed_joint" type="fixed">
-     <parent link="wrist_3_link" />
-     <child link = "ee_link" />
-     <origin xyz="0.0 0.0 0.0" rpy="0.0 0.0 ${pi/2.0}" />
-   </joint>
-   <link name="ee_link">
-     <!-- <collision>
-       <geometry>
-         <box size="0.01 0.01 0.01"/>
-       </geometry>
-       <origin rpy="0 0 0" xyz="-0.01 0 0"/>
-     </collision>
-     <visual>
-       <geometry>
-         <box size="0.01 0.01 0.01"/>
-       </geometry>
-       <origin rpy="0 0 0" xyz="-0.01 0 0"/>
-     </visual> -->
-   </link>
-   <link name="ur3e_d435_mount_link">
-     <inertial>
-       <origin xyz="0.0 0.0 0.0" rpy="0 0 0" />
-       <mass value="0.1"/>
-       <inertia ixx="0.001" ixy="0.0" ixz="0.0"
-         iyy="0.001" iyz="0.0"
-         izz="0.001" />
-     </inertial>
-     <visual>
-       <origin xyz="0 0 0" rpy="0 0 0" />
-       <geometry>
-         <mesh filename="package://agimus_demos/ur3/pointing/meshes/ur3e_d435_mount.stl"/>
-       </geometry>
-       <material name="Red">
-         <color rgba="0.9 0.1 0.1 1.0"/>
-       </material>
-     </visual>
-     <collision>
-       <origin xyz="0 0 0" rpy="0 0 0" />
-       <geometry>
-         <mesh filename="package://agimus_demos/ur3/pointing/meshes/ur3e_d435_mount.stl"/>
-       </geometry>
-     </collision>
-   </link>
-   <joint name="ur3e_d435_mount_joint" type="fixed">
-     <parent link="wrist_3_link"/>
-     <child link="ur3e_d435_mount_link" />
-     <origin xyz="0.0 0.0 0.0" rpy="0.0 0.0 3.14159265359" />
-   </joint>
-   <link name="ur3e_tool_link">
-     <inertial>
-       <origin xyz="0.0 0.0 0.0" rpy="0 0 0" />
-       <mass value="0.1"/>
-       <inertia ixx="0.001" ixy="0.0" ixz="0.0"
-         iyy="0.001" iyz="0.0"
-         izz="0.001" />
-     </inertial>
-     <!-- Tool support -->
-     <visual>
-       <origin xyz="0 0 0" rpy="0 0 0" />
-       <geometry>
-         <mesh filename="package://agimus_demos/ur3/pointing/meshes/ur3e_tip.stl"/>
-       </geometry>
-       <material name="Red">
-         <color rgba="0.9 0.1 0.1 1.0"/>
-       </material>
-     </visual>
-     <collision>
-       <origin xyz="0 0 0" rpy="0 0 0" />
-       <geometry>
-         <mesh filename="package://agimus_demos/ur3/pointing/meshes/ur3e_tip.stl"/>
-       </geometry>
-     </collision>
-     <!-- wooden spike -->
-     <visual>
-       <origin xyz="0 0 0.113" rpy="0 0 0" />
-       <geometry>
-	 <cylinder radius="0.0015" length="0.25"/>
-       </geometry>
-       <material name="Pine">
-	 <color rgba="0.8 0.65 0.4 1.0"/>
-       </material>
-     </visual>
-     <collision>
-       <origin xyz="0 0 0.113" rpy="0 0 0" />
-       <geometry>
-	 <cylinder radius="0.0015" length="0.25"/>
-       </geometry>
-     </collision>
-   </link>
-   <joint name="ur3e_tool_joint" type="fixed">
-     <parent link="ur3e_d435_mount_link"/>
-     <child link="ur3e_tool_link" />
-     <origin xyz="$(arg tip_offset_x) $(arg tip_offset_y) 0.0" rpy="0.0 0.0 0.0" />
-   </joint>
-   <link name="ur3e_tooltip_link">
-   </link>
-  <joint name="ur3e_tooltip_joint" type="fixed">
-     <parent link="ur3e_tool_link" />
-     <child link = "ur3e_tooltip_link" />
-     <origin xyz="0.0 0.0 ${0.25 + $(arg tip_offset_z)}" rpy="0.0 0.0 0.0" />
-  </joint>
    <link name="ref_camera_link">
    </link>
     <joint name="ref_camera_joint" type="fixed">
-     <parent link="ur3e_d435_mount_link" />
+     <parent link="wrist_3_link" />
      <child link = "ref_camera_link" />
      <origin xyz="${camera_pose['camera']['x']}

Commit message: add gripper model + graph constraint update

File: ur3/pointing/urdf/robot.urdf.xacro (robot description, xacro)
@@ -86,11 +86,11 @@
      <link name="walls">
      <!-- front wall -->
-     <visual>
-	<origin xyz="0.385 -0.305 0.37"/>
-        <geometry>
-	  <box size="0.03 1 0.74"/>
-        </geometry>
-	<material name="white02"/>
-     </visual>
+     <!-- visual -->
+	<!-- origin xyz="0.385 -0.305 0.37"/ -->
+        <!-- geometry -->
+	  <!-- box size="0.03 1 0.74"/ -->
+        <!-- /geometry -->
+	<!-- material name="white02"/ -->
+     <!-- /visual -->
       <collision>
        <origin xyz="0.385 -0.305 0.37"/>
@@ -171,23 +171,31 @@
       <origin xyz="0.0 0.0 1" rpy="0.0 0.0 -1.5707963" />
    </joint>
-   <link name="collision_cylinder">
-     <visual>
-        <origin xyz="0 0 0" rpy="0 0 0"/>
-       <geometry>
-	 <cylinder radius="0.045" length="0.115"/>
-       </geometry>
-     </visual>
-     <collision>
-       <origin xyz="0 0 0" rpy="0 0 0"/>
-       <geometry>
-	 <cylinder radius="0.045" length="0.115"/>
-       </geometry>
-     </collision>
-   </link>
-   <joint name="collision_cylinder_joint" type="fixed">
-     <parent link="wrist_3_link" />
-     <child link = "collision_cylinder" />
-     <origin xyz="0.0 0.0 0.05" rpy="0.0 0.0 ${pi/2.0}" />
-   </joint>
+    <link name="ee_gripper">
+      <visual>
+        <geometry>
+          <!-- The path to the visual meshes in the package. -->
+          <mesh filename="package://agimus_demos/ur3/pointing/meshes/gripper_2f85_opened.stl" scale = "0.0008 0.0008 0.0008" />
+        </geometry>
+      </visual>
+      <collision>
+        <geometry>
+          <!-- The path to the collision meshes in the package. -->
+          <mesh filename="package://agimus_demos/ur3/pointing/meshes/gripper_2f85_opened.stl" scale = "0.0008 0.0008 0.0008" />
+        </geometry>
+      </collision>
+    </link>
+    <joint name="ee_gripper_joint" type="fixed">
+      <!-- The parent link must be read from the robot model it is attached to. -->
+      <parent link="wrist_3_link"/>
+      <child link="ee_gripper"/>
+      <origin rpy="1.5708 0 0" xyz="0 0.075 0"/>
+    </joint>
+    <!-- TCP frame -->
+    <joint name="tcp_joint" type="fixed">
+      <origin xyz="0 0 0.116" rpy="0 0 0"/>
+      <parent link="ee_gripper"/>
+      <child link="tcp"/>
+    </joint>
+    <link name="tcp"/>
    <link name="ref_camera_link">
    </link>

Commit message: upload robotiq gripper urdf

File: ur3/pointing/urdf/robot.urdf.xacro (robot description, xacro)
@@ -19,5 +19,5 @@
        - hardware_interface/VelocityJointInterface
        - hardware_interface/EffortJointInterface
-  -->
+-->
   <xacro:arg name="transmission_hw_interface"
              default="hardware_interface/PositionJointInterface"/>
@@ -171,31 +171,57 @@
       <origin xyz="0.0 0.0 1" rpy="0.0 0.0 -1.5707963" />
    </joint>
-    <link name="ee_gripper">
-      <visual>
-        <geometry>
-          <!-- The path to the visual meshes in the package. -->
-          <mesh filename="package://agimus_demos/ur3/pointing/meshes/gripper_2f85_opened.stl" scale = "0.0008 0.0008 0.0008" />
-        </geometry>
-      </visual>
-      <collision>
-        <geometry>
-          <!-- The path to the collision meshes in the package. -->
-          <mesh filename="package://agimus_demos/ur3/pointing/meshes/gripper_2f85_opened.stl" scale = "0.0008 0.0008 0.0008" />
-        </geometry>
-      </collision>
+    <!-- End Effector -->
+    <joint name="ee_fixed_joint" type="fixed">
+        <parent link="wrist_3_link"/>
+        <child link="ee_link"/>
+        <origin rpy="0.0 0.0 1.57079632679" xyz="0.0 0.0823 0.0"/>
+    </joint>
+    <link name="ee_link">
+    <collision>
+      <geometry>
+        <box size="0.01 0.01 0.01"/>
+      </geometry>
+      <origin rpy="0 0 0" xyz="-0.01 0 0"/>
+    </collision>
     </link>
-    <joint name="ee_gripper_joint" type="fixed">
-      <!-- The parent link must be read from the robot model it is attached to. -->
-      <parent link="wrist_3_link"/>
-      <child link="ee_gripper"/>
-      <origin rpy="1.5708 0 0" xyz="0 0.075 0"/>
-    </joint>
-    <!-- TCP frame -->
-    <joint name="tcp_joint" type="fixed">
-      <origin xyz="0 0 0.116" rpy="0 0 0"/>
-      <parent link="ee_gripper"/>
-      <child link="tcp"/>
-    </joint>
-    <link name="tcp"/>
+  <!-- Robotiq Coupler -->
+  <!-- Gripper -->
+  <xacro:include filename="$(find agimus_demos)/ur3/pointing/urdf/robotiq_gripper/robotiq_85_gripper.urdf.xacro" />
+  <!--  + Height added by the coupler: 8mm -->
+  <!--  + Reference frame: at the middle (4mm) -->
+  <link name="robotiq_coupler">
+    <visual>
+      <geometry>
+        <mesh filename="package://agimus_demos/ur3/pointing/meshes/robotiq_85_coupler.stl" />
+      </geometry>
+      <material name="flat_black"/>
+    </visual>
+    <collision>
+      <geometry>
+        <mesh filename="package://agimus_demos/ur3/pointing/meshes/robotiq_85_coupler.stl" />
+      </geometry>
+    </collision>
+    <inertial>
+      <origin xyz="2.073e-05   1.45286e-03  -1.1049e-03" rpy="0 0 0" />
+      <mass value="0.168" />
+      <inertia ixx="6.69695624e-05" ixy="5.21511788e-09" ixz="-2.74383009e-08"
+               iyy="7.85088161e-05" iyz="5.41105193e-07" izz="1.41819717e-04"/>
+    </inertial>
+  </link>
+  <joint name="robotiq_coupler_joint" type="fixed">
+    <origin xyz="0 0 0.004" rpy="0 0 ${-pi/2.0}" />
+    <parent link="tool0"/>
+    <child link="robotiq_coupler"/>
+  </joint>
+  <gazebo reference="robotiq_coupler">
+    <mu1>0.9</mu1>
+    <mu2>0.9</mu2>
+    <material>Gazebo/FlatBlack</material>
+  </gazebo>
+  <!-- Attach the robotiq 85 gripper -->
+  <xacro:robotiq_85_gripper prefix="" parent="robotiq_coupler" >
+    <origin xyz="0 0 0.004" rpy="0 ${-pi/2} ${pi}"/>
+  </xacro:robotiq_85_gripper>
+   <!-- Camera -->
    <link name="ref_camera_link">
    </link>

File: urdf/d435_gazebo.urdf.xacro (robot description, xacro)
@@ -7,4 +7,17 @@
       <!--robotSimType>gazebo_ros_control/DefaultRobotHWSim</robotSimType-->
     </plugin>
+  </gazebo>
+  <!-- Gazebo grasping plugin -->
+  <gazebo>
+    <gripper name="gazebo_gripper">
+      <grasp_check>
+        <attach_steps>2</attach_steps>    <!-- default: 20 -->
+        <detach_steps>2</detach_steps>    <!-- default: 40 -->
+        <min_contact_count>3</min_contact_count>
+      </grasp_check>
+      <gripper_link>robotiq_85_left_finger_tip_link</gripper_link>
+      <gripper_link>robotiq_85_right_finger_tip_link</gripper_link>
+      <palm_link>robotiq_85_base_link</palm_link>
+    </gripper>
   </gazebo>
   <xacro:include filename="$(find agimus_demos)/urdf/_d435.gazebo.xacro"/>
